File: ICEBATS384/FPGA.kicad_sch (KiCad schematic)
At the start: 11 parts, among them U1 ICE40LP384-SG32

Commit message: Sheet documentation
Other:
- company: (none) -> Soldersplash
- title: (none) -> ICEBATS384
Changed lines of the file:
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@@
 	(generator_version "9.0")
 	(paper "A4")
+	(title_block
+		(title "ICEBATS384")
+		(date "2025-06-13")
+		(rev "A")
+		(company "Soldersplash")
+	)
 	(junction
 		(at 77.47 72.39)
