File: ICEBATS384/Flash.kicad_sch (KiCad schematic)
At the start: 3 parts, among them U2 W25X40CLUXIG TR

Commit message: Fixes missing schematic connections.
Parts:
- removed C8: 110nF, Capacitor_SMD:C_0402_1005Metric, symbol Device:C_Small
- removed R4: 10k, Resistor_SMD:R_0402_1005Metric, symbol Device:R_Small
- removed U2: W25X40CLUXIG TR, Package_SON:Winbond_USON-8-1EP_3x2mm_P0.5mm_EP0.2x1.6mm, symbol 2025-06-09_04-19-34:W25X40CLUXIG_TR
Changed lines of the file:
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@@
 	(generator_version "9.0")
 	(paper "A4")
+)

Commit message: Sheet documentation
Other:
- title: (none) -> ICEBATS384
Changed lines of the file:
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@@
 	(generator_version "9.0")
 	(paper "A4")
+	(title_block
+		(title "ICEBATS384")
+		(date "2025-06-13")
+		(rev "A")
+	)
 )
