File: ICEBATS384/Indicators.kicad_sch (KiCad schematic)
At the start: 10 parts

Commit message: Sheet documentation
Other:
- company: (none) -> Soldersplash
- title: (none) -> ICEBATS384
Changed lines of the file:
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@@
 	(generator_version "9.0")
 	(paper "A4")
+	(title_block
+		(title "ICEBATS384")
+		(date "2025-06-13")
+		(rev "A")
+		(company "Soldersplash")
+	)
 	(wire
 		(pts
